File: hardware/watch/watch.kicad_sch (KiCad schematic)
At the start: 0 parts

Commit message: Switch to local project library
Parts:
- added U?: STM32WB55CGU6TR, symbol snoopy:STM32WB55CGU6TR
Connections:
- new net SCL: U?.5 (PB8)
- new net SDA: U?.6 (PB9)
Changed lines of the file:
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@@
-(kicad_sch (version 20211123) (generator eeschema)
+(kicad_sch (version 20230121) (generator eeschema)
   (paper "A4")
+  (label "SDA" (at 261.62 68.58 0) (fields_autoplaced)
+    (effects (font (size 1.27 1.27)) (justify left bottom))
+  )
+  (label "SCL" (at 261.62 66.04 0) (fields_autoplaced)
+    (effects (font (size 1.27 1.27)) (justify left bottom))
+  )
+  (symbol (lib_id "snoopy:STM32WB55CGU6TR") (at 241.3 86.36 0) (unit 1)
+    (in_bom yes) (on_board yes) (dnp no) (fields_autoplaced)
+    (property "Reference" "U?" (at 241.3 34.29 0)
+      (effects (font (size 1.27 1.27)))
+    )
+    (property "Value" "STM32WB55CGU6TR" (at 241.3 121.92 0)
+      (effects (font (size 1.27 1.27)) hide)
+    )
+    (property "Footprint" "" (at 241.3 124.46 0)
+      (effects (font (size 1.27 1.27)) hide)
+    )
+    (property "Datasheet" "https://www.st.com/resource/en/datasheet/stm32wb55cc.pdf" (at 241.3 127 0)
+      (effects (font (size 1.27 1.27)) hide)
+    )
+    (property "Name" "STM32WB55CGU6TR" (at 241.3 36.83 0)
+      (effects (font (size 1.27 1.27)))
+    )
+    (property "Link (DigiKey)" "https://www.digikey.com/en/products/detail/stmicroelectronics/STM32WB55CGU6TR/10326853" (at 241.3 139.7 0)
+      (effects (font (size 1.27 1.27)) hide)
+    )
+    (property "Identifier (DigiKey)" "497-STM32WB55CGU6TRCT-ND" (at 241.3 137.16 0)
+      (effects (font (size 1.27 1.27)) hide)
+    )
+    (property "Description (DigiKey)" "IC RF TxRx + MCU 802.15.4, Bluetooth Bluetooth v5.3, Thread, Zigbee® 2.405GHz ~ 2.48GHz 48-UFQFN Exposed Pad Cut Tape" (at 241.3 129.54 0)
+      (effects (font (size 1.27 1.27)) hide)
+    )
+    (pin "1")
+    (pin "10")
+    (pin "11")
+    (pin "12")
+    (pin "13")
+    (pin "14")
+    (pin "15")
+    (pin "16")
+    (pin "17")
+    (pin "18")
+    (pin "19")
+    (pin "2")
+    (pin "20")
+    (pin "21")
+    (pin "22")
+    (pin "23")
+    (pin "24")
+    (pin "25")
+    (pin "26")
+    (pin "27")
+    (pin "28")
+    (pin "29")
+    (pin "3")
+    (pin "30")
+    (pin "31")
+    (pin "32")
+    (pin "33")
+    (pin "34")
+    (pin "35")
+    (pin "36")
+    (pin "37")
+    (pin "38")
+    (pin "39")
+    (pin "4")
+    (pin "40")
+    (pin "41")
+    (pin "42")
+    (pin "43")
+    (pin "44")
+    (pin "45")
+    (pin "46")
+    (pin "47")
+    (pin "48")
+    (pin "5")
+    (pin "6")
+    (pin "7")
+    (pin "8")
+    (pin "9")
+    (instances
+      (project "watch"
+        (path "/90f1d9be-2356-4bcc-9cf9-80f751451366"
+          (reference "U?") (unit 1)
+        )
+      )
+    )
+  )
   (sheet_instances
     (path "/" (page "1"))
